Commit message: 调整tf变换树

File: How_to_change_urdf_model/turtlebot3_burger.urdf.xacro (robot description, xacro)
@@ -116,10 +116,9 @@
     <parent link="base_link"/>
     <child link="base_kinect2"/>
-    <origin xyz="-0.012 0 0.152" rpy="0 0 0"/>
+    <origin xyz="-0.012 0 0.172" rpy="0 0 0"/>
   </joint>
   <link name="base_kinect2">
     <visual>
-      <!-- <origin xyz="0.02 0 -0.03" rpy="0 0 -1.57075"/> -->
-      <origin xyz="0 0 0.0" rpy="0 0 -1.57075"/>
+      <origin xyz="0 0 -0.03" rpy="0 0 -1.57075"/>
       <geometry>
         <mesh filename="package://turtlebot3_description/meshes/sensors/Kinect2.stl" scale="0.001 0.001 0.001"/>
@@ -144,9 +143,8 @@
     <parent link="base_link"/>
     <child link="base_vlc_mvcam"/>
-    <origin xyz="0.062 0 0.088" rpy="0 0 0"/>
+    <origin xyz="0.060 0 0.105" rpy="0 0 0"/>
   </joint>
   <link name="base_vlc_mvcam">
     <visual>
-      <!-- <origin xyz="0.09 0 -0.03" rpy="0 0 0"/> -->
       <origin xyz="0.0 0 -0.03" rpy="0 0 0"/>
       <geometry>

Commit message: 更新了仅加入mvcam的turtlebot3模型urdf

File: How_to_change_urdf_model/turtlebot3_burger.urdf.xacro (robot description, xacro)
@@ -110,17 +110,17 @@
     <parent link="base_link"/>
     <child link="imu_link"/>
-    <origin xyz="-0.032 0 0.068" rpy="0 0 3.1415"/>
+    <origin xyz="-0.032 0 0.068" rpy="0 0 3.141526"/>
   </joint>
   <link name="imu_link"/>
   <joint name="scan_joint" type="fixed">
     <parent link="base_link"/>
-    <child link="base_kinect2"/>
-    <origin xyz="-0.012 0 0.172" rpy="0 0 0"/>
+    <child link="base_scan"/>
+    <origin xyz="-0.032 0 0.172" rpy="0 0 0"/>
   </joint>
-  <link name="base_kinect2">
+  <link name="base_scan">
     <visual>
-      <origin xyz="0 0 -0.03" rpy="0 0 -1.57075"/>
+      <origin xyz="0 0 0.0" rpy="0 0 0"/>
       <geometry>
-        <mesh filename="package://turtlebot3_description/meshes/sensors/Kinect2.stl" scale="0.001 0.001 0.001"/>
+        <mesh filename="package://turtlebot3_description/meshes/sensors/lds.stl" scale="0.001 0.001 0.001"/>
       </geometry>
       <material name="dark"/>
