Commit message: 明确了定位结果为相机镜头外侧镜片中心所在的位置

File: How_to_edit_urdf_model/turtlebot3_burger.urdf.xacro (robot description, xacro)
@@ -143,9 +143,9 @@
     <parent link="base_link"/>
     <child link="base_vlc_mvcam"/>
-    <origin xyz="0.060 0 0.105" rpy="0 0 0"/>
+    <origin xyz="0.060 0 0.155" rpy="0 0 0"/>
   </joint>
   <link name="base_vlc_mvcam">
     <visual>
-      <origin xyz="0.0 0 -0.03" rpy="0 0 0"/>
+      <origin xyz="0.0 0 -0.08" rpy="0 0 0"/>
       <geometry>
         <mesh filename="package://turtlebot3_description/meshes/sensors/mvcam.stl" scale="0.001 0.001 0.001"/>
